Commit message: Enable other packages to use provided urdfs

File: urdf/realsense-RS200.macro.xacro (robot description, xacro)
@@ -17,5 +17,5 @@
             <origin rpy="0 0 0" xyz="0 0 0"/>
             <geometry>
-                <mesh filename="package://realsense_gazebo_plugin/models/realsense_camera/meshes/realsense.dae"/>
+                <mesh filename="$(find realsense_gazebo_plugin)/models/realsense_camera/meshes/realsense.dae"/>
             </geometry>
         </visual>
